File: clock_design.kicad_pcb (KiCad board)
At the start: 2 copper layers, 118 x 118 mm, 107 parts, among them J1 Power_inlet_vertical, J2 Conn_01x06, J3 Conn_01x03, J4 Conn_01x03, J5 Conn_02x03_Odd_Even, SW1 Omron_B3F_SPST, SW2 Omron_B3F_SPST, SW3 Omron_B3F_SPST, SW4 Omron_B3F_SPST, SW5 Omron_B3F_SPST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

Commit message: Routing in progress...
Parts:
- added D4: LED_0805_GRN, footprints:LED_0805_2012Metric, F.Cu at (203.2, 90.2)
- added R17: R_0805_2.2K, footprints:R_0805_2012Metric, F.Cu at (196.8, 90.2)
- C10, C11, C13, C16, C17, C22, C23, C24, C4, C5, C8, C9, R16, R3, R7, R8: moved to B.Cu
- moved C10 241.5 mm to (141.0, 96.9), turned to 90 degrees
- moved R3 237.8 mm to (135.9, 96.5), turned to 90 degrees
- moved C11 234.5 mm to (143.5, 97.3), turned to 90 degrees
- moved R13 230.2 mm to (105.4, 115.6)
- moved R12 225.2 mm to (96.5, 91.4)
- moved C17 220.5 mm to (118.5, 123.2), turned to 180 degrees
- moved R18 219.8 mm to (109.2, 137.2)
- moved C4 216.9 mm to (161.3, 113.0), turned to -90 degrees
- moved C22 212.2 mm to (117.1, 120.7), turned to 180 degrees
- moved C8 210.4 mm to (166.4, 113.0), turned to -90 degrees
- moved C24 207.2 mm to (138.4, 96.9), turned to 90 degrees
- moved R11 204.6 mm to (142.2, 154.9)
- moved R8 190.9 mm to (151.1, 144.8), turned to 180 degrees
- moved R16 188.4 mm to (154.9, 81.3), turned to 180 degrees
- moved R7 183.7 mm to (151.1, 142.2)
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Routing:
- net SPI_MOSI: track 0.00 -> 207.5 mm, vias 0 -> 2
- net SPI_MISO: track 0.00 -> 187.9 mm, vias 0 -> 2
- net SPI_SCLK: track 0.00 -> 162.7 mm, vias 0 -> 1
- net SEG_E: track 0.00 -> 124.2 mm, vias 0 -> 1
- net BUTTON_MODE_L: track 0.00 -> 115.0 mm, vias 0 -> 2
- net RESET_L: track 0.00 -> 107.3 mm, vias 0 -> 3
- net SEG_B: track 0.00 -> 96.3 mm, vias 0 -> 1
- net SEG_A: track 0.00 -> 80.8 mm, vias 0 -> 1
- net SEG_G: track 0.00 -> 77.3 mm, vias 0 -> 1
- net SEG_F: track 0.00 -> 74.8 mm, vias 0 -> 1
- net SEG_D: track 0.00 -> 73.7 mm, vias 0 -> 1
- net SEG_C: track 0.00 -> 68.2 mm, vias 0 -> 2
- net SEG_DP: track 0.00 -> 62.3 mm
- net UART_RX: track 0.00 -> 53.3 mm, vias 0 -> 1
- net UART_TX: track 0.00 -> 52.1 mm, vias 0 -> 1
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- added copper zone on F.Cu, net GND
- added copper zone on B.Cu, net PP5V0

Commit message: Initial gerber out
Got all of the files for gereber out
Parts:
- removed C14, C15, C18, C21: C_0805_0.1uf, footprints:C_0805_2012Metric
- removed the R17 at (321.7, 86.9)
- removed R19: R_0805_4.7K, footprints:R_0805_2012Metric
- removed TP10, TP11, TP12, TP13, TP14, TP15, TP16, TP17, TP18, TP19, TP20, TP21, TP3, TP4, TP5, TP6, TP7, TP8, TP9: TestPoint, footprints:TestPoint_THTPad_D2.0mm_Drill1.0mm
- C1, R14, R2, R22, R23, R4, TP1, TP25: moved to B.Cu
- R6: moved to F.Cu
- moved C12 270.7 mm to (101.7, 121.3), turned to 90 degrees
- moved R4 242.8 mm to (125.4, 86.7), turned to 180 degrees
- moved R5 236.9 mm to (109.1, 128.8), turned to 180 degrees
- moved R21 229.8 mm to (116.8, 138.4)
- moved R2 222.6 mm to (125.5, 84.5), turned to 180 degrees
- moved R1 186.3 mm to (171.4, 120.7), turned to 180 degrees
- moved C1 173.5 mm to (188.0, 115.6), turned to -90 degrees
- moved TP1 166.2 mm to (189.2, 104.1), turned to 180 degrees
- moved TP25 160.4 mm to (188.0, 127.7), turned to 180 degrees
- moved TP2 149.3 mm to (191.8, 94.0)
- moved R20 141.3 mm to (189.2, 81.4), turned to 180 degrees
- moved R23 123.1 mm to (189.2, 87.6), turned to 180 degrees
- moved TP22 122.9 mm to (157.1, 110.1)
- moved R22 115.6 mm to (189.2, 85.1), turned to 180 degrees
- moved TP23 99.8 mm to (134.6, 113.4)
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Connections:
- U1 pad 6: DEBUG_LED_0 -> DEBUG_LED_1
Routing:
- net SPI_MATRIX_SS_L: track 0.00 -> 127.8 mm, vias 0 -> 2
- net BUTTON_HOURS_L: track 15.2 -> 128.8 mm, vias 0 -> 4
- net ADC_0: track 0.00 -> 112.6 mm, vias 0 -> 2
- net DEBUG_LED_1: track 0.00 -> 90.8 mm, vias 0 -> 1
- net DEBUG_LED_0: track 0.00 -> 82.5 mm, vias 0 -> 1
- net SPI_DIG_DISPLAY_SS_L: track 0.00 -> 80.0 mm, vias 0 -> 2
- net Net-(J4-Pad3): track 0.00 -> 65.5 mm, vias 0 -> 3
- net BUTTON_MINUTES_L: track 0.00 -> 61.9 mm, vias 0 -> 2
- net MATRIX_ROW_6: track 0.00 -> 61.2 mm, vias 0 -> 1
- net Net-(BT1-Pad1): track 0.00 -> 61.1 mm
- net MATRIX_COL_2: track 0.00 -> 59.0 mm, vias 0 -> 1
- net SEG_A: track 80.8 -> 138.9 mm
- net MATRIX_ROW_5: track 0.00 -> 51.3 mm, vias 0 -> 1
- net MATRIX_COL_3: track 0.00 -> 50.8 mm, vias 0 -> 4
- net MATRIX_ROW_3: track 0.00 -> 46.3 mm, vias 0 -> 2
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- added copper zone on B.Cu, net GND
- added copper zone on F.Cu, net PP5V0
Other:
- board text added: ":"
- board text added: "Ershov time"
